File: led-module.brd (EAGLE design)
At the start: 40 x 80 mm, 36 parts, among them U1 LT3956EUHEPBFUHE_36_ADI-M, U2 RUR020N02TL

Commit message: Added libraries
Parts:
- removed H1, H2, H3, H4: MOUNT-HOLE5.0, holes:5,0
- moved U$1 19.9 mm to (20.0, 40.0)
Routing:
- net N$7: track 32.2 -> 51.8 mm
Changed lines of the file:
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@@
 <attribute name="VALUE" x="16.97" y="20.59" size="1.27" layer="27" rot="R270"/>
 </element>
-<element name="U$1" library="5-2154874-3" package="5-2154874-3" value="5-2154874-3" x="20.062" y="59.888" smashed="yes" rot="R180"/>
-<element name="H1" library="holes" library_urn="urn:adsk.eagle:library:237" package="5,0" package3d_urn="urn:adsk.eagle:package:14276/1" value="MOUNT-HOLE5.0" x="34.655" y="4.916" smashed="yes">
-<attribute name="POPULARITY" value="0" x="34.655" y="4.916" size="1.778" layer="27" display="off"/>
-</element>
-<element name="H2" library="holes" library_urn="urn:adsk.eagle:library:237" package="5,0" package3d_urn="urn:adsk.eagle:package:14276/1" value="MOUNT-HOLE5.0" x="35.874" y="74.939" smashed="yes">
-<attribute name="POPULARITY" value="0" x="35.874" y="74.939" size="1.778" layer="27" display="off"/>
-</element>
-<element name="H3" library="holes" library_urn="urn:adsk.eagle:library:237" package="5,0" package3d_urn="urn:adsk.eagle:package:14276/1" value="MOUNT-HOLE5.0" x="19.097" y="44.903" smashed="yes">
-<attribute name="POPULARITY" value="0" x="19.097" y="44.903" size="1.778" layer="27" display="off"/>
-</element>
-<element name="H4" library="holes" library_urn="urn:adsk.eagle:library:237" package="5,0" package3d_urn="urn:adsk.eagle:package:14276/1" value="MOUNT-HOLE5.0" x="35.536" y="30.421" smashed="yes">
-<attribute name="POPULARITY" value="0" x="35.536" y="30.421" size="1.778" layer="27" display="off"/>
-</element>
+<element name="U$1" library="5-2154874-3" package="5-2154874-3" value="5-2154874-3" x="20" y="40" smashed="yes" rot="R180"/>
 </elements>
 <signals>
@@
 <wire x1="22.1056" y1="20.63369375" x2="20.16169375" y2="22.5776" width="0.3" layer="16"/>
 <wire x1="20.16169375" y1="22.5776" x2="18.7224" y2="22.5776" width="0.3" layer="16"/>
-<wire x1="5.469890625" y1="75.323890625" x2="4.822" y2="76.398" width="0" layer="19" extent="1-1"/>
+<wire x1="5.469890625" y1="75.323890625" x2="4.76" y2="56.51" width="0" layer="19" extent="1-1"/>
 </signal>
 <signal name="N$14">
@@
 <wire x1="18.167" y1="37.24" x2="31.816" y2="37.24" width="2" layer="1"/>
 <wire x1="35.302" y1="40.726" x2="31.816" y2="37.24" width="2" layer="1"/>
-<wire x1="35.302" y1="40.726" x2="35.302" y2="40.838" width="2" layer="1"/>
+<wire x1="35.302" y1="40.726" x2="35.24" y2="20.95" width="2" layer="1"/>
 </signal>
 <signal name="N$15">

Commit message: Layout wip
Parts:
- removed JP2: (no value), pinhead:1X01
- removed JP3: (no value), pinhead:1X02
- removed TP1, TP2, TP3: TPSTP20SQ, testpad:TP20SQ
- JP1: device pinhead:1X02 -> pinhead:1X06
- moved TP4 40.8 mm to (56.6, 34.3)
- moved JP1 34.1 mm to (37.3, 8.86)
- moved C1 28.9 mm to (34.1, 6.14), turned to 90 degrees
- moved C5 28.4 mm to (5.20, 17.8), turned to 180 degrees
- moved R10 27.2 mm to (3.84, 15.7), turned to 180 degrees
- moved C4 26.6 mm to (7.16, 10.9), turned to 270 degrees
- moved R11 25.9 mm to (5.04, 16.7), turned to 0 degrees
- moved R4 24.7 mm to (8.21, 10.8), turned to 90 degrees
- moved R3 24.6 mm to (6.76, 15.2), turned to 0 degrees
- moved C2 24.4 mm to (32.0, 6.17), turned to 90 degrees
- moved C3 23.9 mm to (11.4, 11.0), turned to 90 degrees
- moved R5 23.3 mm to (7.72, 17.8), turned to 0 degrees
- moved R8 22.6 mm to (9.26, 10.8), turned to 270 degrees
- moved R9 22.6 mm to (10.3, 10.8), turned to 90 degrees
- moved R6 15.9 mm to (26.1, 21.9), turned to 0 degrees
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Connections:
- removed net N$13: JP2.1, U1.33
- removed net N$2: C1.1, C2.1, JP1.2, L1.2, R10.2, R8.2, TP1.TP, U1.6
- removed net N$7: JP3.2, TP4.TP, U$1.P$2, U2.3
- new net LED-: TP4.TP, U$1.P$2, U2.3
- new net LED_ON: JP1.4, U1.33
- new net VIN: C1.1, C2.1, JP1.5, JP1.6, L1.2, R10.2, R8.2, U1.6
- net GND: now also JP1.2; no longer TP2.TP
- net ISN: no longer JP3.1, TP3.TP
Routing:
- net ISN: track 79.3 -> 0.00 mm, vias 1 -> 0
- net VIN: track 0.00 -> 65.7 mm, vias 0 -> 3
- net N$2: track 54.8 -> 0.00 mm, vias 3 -> 0
- net N$7: track 51.8 -> 0.00 mm
- net LED_ON: track 0.00 -> 37.9 mm, vias 0 -> 1
- net ISP: track 21.7 -> 0.00 mm, vias 2 -> 0
- net N$3: track 3.60 -> 22.6 mm, vias 0 -> 2
- net N$13: track 9.61 -> 0.00 mm
- net N$12: track 25.2 -> 19.8 mm
- net GND: track 26.1 -> 30.9 mm, vias 122 -> 32
- net N$16: track 3.29 -> 6.09 mm
- net N$9: track 3.56 -> 1.70 mm
- net N$15: track 5.01 -> 3.46 mm
- net N$5: track 2.62 -> 3.72 mm
- net N$1: track 10.5 -> 11.3 mm
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- added copper zone on layer 1, net VIN
- removed copper zone on layer 1, net ISP

Commit message: Sent to production files
Parts:
- removed TP4: TPSTP20SQ, testpad:TP20SQ
- R6: value 250m -> 0.250; device rcl:R0805W -> rcl:WSC2515
- moved R6 10.1 mm to (18.9, 29.0), turned to 180 degrees
Connections:
- net LED-: no longer TP4.TP
Routing:
- net ISN: track 0.00 -> 55.2 mm
- net ISP: track 0.00 -> 41.1 mm, vias 0 -> 2
- net LED-: track 0.00 -> 9.44 mm
- net GND: vias 32 -> 95
