File: led-module.sch (EAGLE design)
At the start: 36 parts, among them U1 LT3956EUHEPBFUHE_36_ADI-M, U2 RUR020N02TL

Commit message: Added libraries
Parts:
- removed H1, H2, H3, H4: MOUNT-HOLE5.0, holes:MOUNT-HOLE5.0
Changed lines of the file:
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@@
 <part name="C6" library="rcl" library_urn="urn:adsk.eagle:library:334" deviceset="C-EU" device="C0805" package3d_urn="urn:adsk.eagle:package:23617/2" value="10uF"/>
 <part name="U$1" library="5-2154874-3" deviceset="5-2154874-3" device=""/>
-<part name="H1" library="holes" library_urn="urn:adsk.eagle:library:237" deviceset="MOUNT-HOLE" device="5.0" package3d_urn="urn:adsk.eagle:package:14276/1"/>
-<part name="H2" library="holes" library_urn="urn:adsk.eagle:library:237" deviceset="MOUNT-HOLE" device="5.0" package3d_urn="urn:adsk.eagle:package:14276/1"/>
-<part name="H3" library="holes" library_urn="urn:adsk.eagle:library:237" deviceset="MOUNT-HOLE" device="5.0" package3d_urn="urn:adsk.eagle:package:14276/1"/>
-<part name="H4" library="holes" library_urn="urn:adsk.eagle:library:237" deviceset="MOUNT-HOLE" device="5.0" package3d_urn="urn:adsk.eagle:package:14276/1"/>
 </parts>
 <sheets>
@@
 <attribute name="NAME" x="260.096" y="-12.192" size="1.778" layer="95" rot="R90"/>
 </instance>
-<instance part="H1" gate="G$1" x="149.86" y="-78.74" smashed="yes">
-<attribute name="NAME" x="151.892" y="-78.1558" size="1.778" layer="95"/>
-<attribute name="VALUE" x="151.892" y="-81.2038" size="1.778" layer="96"/>
-</instance>
-<instance part="H2" gate="G$1" x="157.48" y="-78.74" smashed="yes">
-<attribute name="NAME" x="159.512" y="-78.1558" size="1.778" layer="95"/>
-<attribute name="VALUE" x="159.512" y="-81.2038" size="1.778" layer="96"/>
-</instance>
-<instance part="H3" gate="G$1" x="165.1" y="-78.74" smashed="yes">
-<attribute name="NAME" x="167.132" y="-78.1558" size="1.778" layer="95"/>
-<attribute name="VALUE" x="167.132" y="-81.2038" size="1.778" layer="96"/>
-</instance>
-<instance part="H4" gate="G$1" x="172.72" y="-78.74" smashed="yes">
-<attribute name="NAME" x="174.752" y="-78.1558" size="1.778" layer="95"/>
-<attribute name="VALUE" x="174.752" y="-81.2038" size="1.778" layer="96"/>
-</instance>
 </instances>

Commit message: Layout wip
Parts:
- removed JP2: (no value), pinhead:PINHD-1X1
- removed JP3: (no value), pinhead:PINHD-1X2
- removed TP1, TP2, TP3: TPSTP20SQ, testpad:TPSTP20SQ
- JP1: device pinhead:PINHD-1X2 -> pinhead:PINHD-1X6
Connections:
- removed net N$13: JP2.1, U1A.PWM
- removed net N$2: C1.1, C2.1, JP1.2, L1.2, R10.2, R8.2, TP1.PP, U1A.VIN
- removed net N$7: JP3.2, TP4.PP, U$1.C, U2.D
- new net LED-: TP4.PP, U$1.C, U2.D
- new net LED_ON: JP1.4, U1A.PWM
- new net VIN: C1.1, C2.1, JP1.5, JP1.6, L1.2, R10.2, R8.2, U1A.VIN
- net GND: now also JP1.2; no longer TP2.PP
- net ISN: no longer JP3.1, TP3.PP

Commit message: Sent to production files
Parts:
- removed TP4: TPSTP20SQ, testpad:TPSTP20SQ
- R6: value 250m -> 0.250; device rcl:R-EU_R0805W -> rcl:R-EU_WSC2515
Connections:
- net LED-: no longer TP4.PP
Changed lines of the file:
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@@
 <part name="C10" library="rcl" library_urn="urn:adsk.eagle:library:334" deviceset="C-EU" device="C0805" package3d_urn="urn:adsk.eagle:package:23617/2" value="10uF"/>
 <part name="U2" library="RUR020N02TL" deviceset="RUR020N02TL" device=""/>
-<part name="TP4" library="testpad" library_urn="urn:adsk.eagle:library:385" deviceset="TPS" device="TP20SQ" package3d_urn="urn:adsk.eagle:package:27980/1"/>
 <part name="U1" library="lt3956" deviceset="LT3956EUHEPBF" device="UHE_36_ADI-M"/>
 <part name="R8" library="rcl" library_urn="urn:adsk.eagle:library:334" deviceset="R-EU_" device="R0402" package3d_urn="urn:adsk.eagle:package:23547/3" value="480k"/>
@@
 <part name="R10" library="rcl" library_urn="urn:adsk.eagle:library:334" deviceset="R-EU_" device="R0402" package3d_urn="urn:adsk.eagle:package:23547/3" value="56.2k"/>
 <part name="R11" library="rcl" library_urn="urn:adsk.eagle:library:334" deviceset="R-EU_" device="R0402" package3d_urn="urn:adsk.eagle:package:23547/3" value="56.2k"/>
-<part name="R6" library="rcl" library_urn="urn:adsk.eagle:library:334" deviceset="R-EU_" device="R0805W" package3d_urn="urn:adsk.eagle:package:23537/2" value="250m"/>
 <part name="C6" library="rcl" library_urn="urn:adsk.eagle:library:334" deviceset="C-EU" device="C0805" package3d_urn="urn:adsk.eagle:package:23617/2" value="10uF"/>
 <part name="U$1" library="5-2154874-3" deviceset="5-2154874-3" device=""/>
 <part name="JP1" library="pinhead" library_urn="urn:adsk.eagle:library:325" deviceset="PINHD-1X6" device="" package3d_urn="urn:adsk.eagle:package:22472/2"/>
+<part name="R6" library="rcl" library_urn="urn:adsk.eagle:library:334" deviceset="R-EU_" device="WSC2515" package3d_urn="urn:adsk.eagle:package:26134/2" value="0.250"/>
 </parts>
 <sheets>
@@
 <attribute name="VALUE" x="237.49" y="-21.59" size="2.54" layer="96" ratio="10" rot="SR0"/>
 </instance>
-<instance part="TP4" gate="G$1" x="231.14" y="-12.7" smashed="yes" rot="R90">
-<attribute name="NAME" x="229.87" y="-13.97" size="1.778" layer="95" rot="R90"/>
-<attribute name="TP_SIGNAL_NAME" x="232.41" y="-11.43" size="1.778" layer="97" rot="R90"/>
-</instance>
 <instance part="U1" gate="A" x="91.44" y="15.24" smashed="yes">
 <attribute name="NAME" x="127.3556" y="21.8186" size="2.0828" layer="95" ratio="6" rot="SR0"/>
@@
 <attribute name="VALUE" x="61.722" y="-54.61" size="1.778" layer="96" rot="R90"/>
 </instance>
+<instance part="C6" gate="G$1" x="213.36" y="-12.7" smashed="yes">
+<attribute name="NAME" x="214.884" y="-12.319" size="1.778" layer="95"/>
+<attribute name="VALUE" x="214.884" y="-17.399" size="1.778" layer="96"/>
+</instance>
+<instance part="U$1" gate="G$1" x="256.54" y="-7.62" smashed="yes">
+<attribute name="NAME" x="260.096" y="-12.192" size="1.778" layer="95" rot="R90"/>
+</instance>
+<instance part="JP1" gate="A" x="-15.24" y="-22.86" smashed="yes" rot="R180">
+<attribute name="NAME" x="-11.43" y="-13.335" size="1.778" layer="95" rot="R180"/>
+<attribute name="VALUE" x="-8.89" y="-12.7" size="1.778" layer="96" rot="R180"/>
+</instance>
 <instance part="R6" gate="G$1" x="220.98" y="-2.54" smashed="yes">
 <attribute name="NAME" x="217.17" y="-1.0414" size="1.778" layer="95"/>
 <attribute name="VALUE" x="217.17" y="-5.842" size="1.778" layer="96"/>
-</instance>
-<instance part="C6" gate="G$1" x="213.36" y="-12.7" smashed="yes">
-<attribute name="NAME" x="214.884" y="-12.319" size="1.778" layer="95"/>
-<attribute name="VALUE" x="214.884" y="-17.399" size="1.778" layer="96"/>
-</instance>
-<instance part="U$1" gate="G$1" x="256.54" y="-7.62" smashed="yes">
-<attribute name="NAME" x="260.096" y="-12.192" size="1.778" layer="95" rot="R90"/>
-</instance>
-<instance part="JP1" gate="A" x="-15.24" y="-22.86" smashed="yes" rot="R180">
-<attribute name="NAME" x="-11.43" y="-13.335" size="1.778" layer="95" rot="R180"/>
-<attribute name="VALUE" x="-8.89" y="-12.7" size="1.778" layer="96" rot="R180"/>
 </instance>
 </instances>
@@
 <junction x="203.2" y="-2.54"/>
 <pinref part="U1" gate="A" pin="ISP"/>
-<pinref part="R6" gate="G$1" pin="1"/>
 <pinref part="C6" gate="G$1" pin="1"/>
 <label x="175.26" y="35.56" size="1.778" layer="95"/>
+<pinref part="R6" gate="G$1" pin="1"/>
 </segment>
 </net>
@@
 <junction x="233.68" y="-2.54"/>
 <pinref part="U1" gate="A" pin="ISN"/>
-<pinref part="R6" gate="G$1" pin="2"/>
 <wire x1="256.54" y1="-5.08" x2="256.54" y2="-2.54" width="0.1524" layer="91"/>
 <wire x1="256.54" y1="-2.54" x2="233.68" y2="-2.54" width="0.1524" layer="91"/>
 <pinref part="U$1" gate="G$1" pin="A"/>
 <label x="175.26" y="30.48" size="1.778" layer="95"/>
+<pinref part="R6" gate="G$1" pin="2"/>
 </segment>
 </net>
@@
 <wire x1="236.22" y1="-10.16" x2="233.68" y2="-10.16" width="0.1524" layer="91"/>
 <wire x1="233.68" y1="-10.16" x2="233.68" y2="-12.7" width="0.1524" layer="91"/>
-<pinref part="TP4" gate="G$1" pin="PP"/>
-<junction x="233.68" y="-12.7"/>
 <wire x1="256.54" y1="-12.7" x2="254" y2="-12.7" width="0.1524" layer="91"/>
 <wire x1="254" y1="-12.7" x2="254" y2="-17.78" width="0.1524" layer="91"/>
